File: rc4.sch (EAGLE design)
At the start: 45 parts, among them IC3 CC2652R1FRGZ, Q1 SI2323DS, Q2 SI2323DS, Y1 Q22FA12800150, Y2 32.768KHz

Commit message: Add files via upload
Parts:
- IC3: device ok-chips-dev:WMCU-CC2652R1FRGZ -> CC2652R1FRGZT:CC2652R1FRGZT
Changed lines of the file:
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@@
 </classes>
 <parts>
-<part name="IC3" library="ok-chips-dev" deviceset="WMCU-CC2652R1FRGZ" device="" value="CC2652R1FRGZ"/>
+<part name="IC3" library="CC2652R1FRGZT" deviceset="CC2652R1FRGZT" device="" value="CC2652R1FRGZ"/>
 <part name="C1" library="ok-discretes-dev" deviceset="CAP" device="-0402" value="100n"/>
 <part name="C2" library="ok-discretes-dev" deviceset="CAP" device="-0402" value="100n"/>
