File: rc4.brd (EAGLE design)
At the start: 29.2 x 41.8 mm, 45 parts, among them IC3 CC2652R1FRGZ, Q1 SI2323DS, Q2 SI2323DS, Y1 Q22FA12800150, Y2 32.768KHz

Commit message: Add files via upload
Parts:
- moved R9 0.09 mm to (17.6, 35.2), turned to 223.1 degrees
Routing:
- net GND: vias 269 -> 270
Changed lines of the file:
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@@
 <setting verticaltext="up"/>
 </settings>
-<grid distance="0.1" unitdist="mm" unit="mm" style="lines" multiple="1" display="yes" altdistance="5" altunitdist="mil" altunit="mm"/>
+<grid distance="0.003125" unitdist="mic" unit="mm" style="lines" multiple="1" display="yes" altdistance="5" altunitdist="mil" altunit="mm"/>
 <layers>
 <layer number="1" name="Top" color="4" fill="1" visible="yes" active="yes"/>
@@
 <wire x1="21.5" y1="10.1" x2="21.5" y2="9.9" width="0.2" layer="25"/>
 <wire x1="21.5" y1="9.9" x2="24.9" y2="9.9" width="0.2" layer="25"/>
+<wire x1="4.89446875" y1="9.6784875" x2="4.89446875" y2="9.833759375" width="0.2" layer="25"/>
+<wire x1="4.89446875" y1="9.833759375" x2="5.751434375" y2="13.980040625" width="0.2" layer="25" curve="-23.355271"/>
+<wire x1="24.88325625" y1="9.84369375" x2="24.88325625" y2="9.975475" width="0.2" layer="25"/>
+<wire x1="24.88325625" y1="9.975475" x2="23.25961875" y2="15.314221875" width="0.2" layer="25" curve="33.831494"/>
 </plain>
 <attributes>
@@
 <attribute name="VALUE" x="21.0153" y="37.751521875" size="0.6096" layer="27" font="vector" ratio="20" rot="SR0" align="top-center"/>
 </element>
-<element name="R9" library="ok-discretes-dev" package="_PKG_C_0402" value="0" x="17.48039375" y="35.219609375" smashed="yes" rot="R270">
-<attribute name="NAME" x="15.746190625" y="34.858565625" size="0.762" layer="25" font="vector"/>
-<attribute name="VALUE" x="16.46439375" y="36.108609375" size="0.508" layer="27" font="vector" rot="R270"/>
+<element name="R9" library="ok-discretes-dev" package="_PKG_C_0402" value="0" x="17.572684375" y="35.2048875" smashed="yes" rot="R223.1">
+<attribute name="NAME" x="16.0191125" y="35.485715625" size="0.762" layer="25" font="vector" rot="R354.4"/>
+<attribute name="VALUE" x="17.5275875" y="36.554159375" size="0.508" layer="27" font="vector" rot="R223.1"/>
 </element>
 <element name="BT1" library="Batteries" package="BATTCON_20MM_4LEGS_OVERPASTE" package3d_urn="urn:adsk.eagle:package:37220/1" value="" x="14.8873" y="9.864" smashed="yes">
@@
 <via x="15.7" y="34.3" extent="1-16" drill="0.2" diameter="0.45"/>
 <via x="16.2" y="34.7" extent="1-16" drill="0.2" diameter="0.45"/>
-<via x="16.7" y="35" extent="1-16" drill="0.2" diameter="0.45"/>
-<via x="16.695928125" y="35.713953125" extent="1-16" drill="0.2" diameter="0.45"/>
+<via x="16.5746125" y="35.12421875" extent="1-16" drill="0.2" diameter="0.45"/>
+<via x="17.0352625" y="35.63919375" extent="1-16" drill="0.2" diameter="0.45"/>
 <via x="17.04034375" y="36.3058625" extent="1-16" drill="0.2" diameter="0.45"/>
 <via x="17.2" y="32.8" extent="1-16" drill="0.2" diameter="0.45"/>
 <via x="17.2" y="33.4" extent="1-16" drill="0.2" diameter="0.45"/>
 <via x="17.4" y="34" extent="1-16" drill="0.2" diameter="0.45"/>
-<via x="18" y="34.3" extent="1-16" drill="0.2" diameter="0.45"/>
-<via x="18.3" y="34.97325625" extent="1-16" drill="0.2" diameter="0.45"/>
-<via x="18.295928125" y="35.681396875" extent="1-16" drill="0.2" diameter="0.45"/>
+<via x="18.07361875" y="34.536965625" extent="1-16" drill="0.2" diameter="0.45"/>
+<via x="18.62309375" y="34.846265625" extent="1-16" drill="0.2" diameter="0.45"/>
+<via x="18.619021875" y="35.6508" extent="1-16" drill="0.2" diameter="0.45"/>
 <via x="14.6" y="32.6" extent="1-16" drill="0.2" diameter="0.45"/>
 <via x="14.1" y="32.9" extent="1-16" drill="0.2" diameter="0.45"/>
@@
 <via x="19.761725" y="33.251965625" extent="1-16" drill="0.2" diameter="0.45"/>
 <via x="20.195465625" y="35.495434375" extent="1-16" drill="0.2" diameter="0.45"/>
-<via x="19.15065" y="35.589578125" extent="1-16" drill="0.2" diameter="0.45"/>
+<via x="19.35080625" y="35.223803125" extent="1-16" drill="0.2" diameter="0.45"/>
 <via x="21.1" y="34.4" extent="1-16" drill="0.2" diameter="0.45"/>
 <via x="19.687240625" y="34.41930625" extent="1-16" drill="0.2" diameter="0.45"/>
@@
 <wire x1="2.4009" y1="26.9036" x2="2.4009" y2="26.871609375" width="0.1524" layer="1"/>
 <wire x1="2.4" y1="26.870709375" x2="2.4009" y2="26.871609375" width="0.1524" layer="1"/>
-<via x="19.024140625" y="36.3" extent="1-16" drill="0.3"/>
+<via x="19.024140625" y="36.3115" extent="1-16" drill="0.3"/>
 <via x="18.51695625" y="36.302825" extent="1-16" drill="0.2" diameter="0.45"/>
 <via x="24.7372125" y="34.40759375" extent="1-16" drill="0.2" diameter="0.45"/>
@@
 <via x="8.3443875" y="29.324521875" extent="1-16" drill="0.2" diameter="0.45"/>
 <via x="7.7443875" y="27.924521875" extent="1-16" drill="0.2" diameter="0.45"/>
+<via x="19.306078125" y="33.591546875" extent="1-16" drill="0.2" diameter="0.45"/>
 </signal>
 <signal name="DCOUPL">
@@
 <contactref element="R9" pad="2"/>
 <contactref element="FL1" pad="1"/>
-<wire x1="15.79" y1="33.5" x2="16.15418125" y2="33.9225125" width="0.254" layer="1"/>
-<wire x1="16.15418125" y1="33.9225125" x2="17.48039375" y2="34.789609375" width="0.3048" layer="1"/>
+<wire x1="17.2587125" y1="34.911078125" x2="16.0974375" y2="33.8074375" width="0.3048" layer="1"/>
+<wire x1="15.79" y1="33.5" x2="16.0974375" y2="33.8074375" width="0.3048" layer="1"/>
 </signal>
 <signal name="N$5">
 <contactref element="R9" pad="1"/>
 <contactref element="E1" pad="ANT"/>
-<wire x1="17.8883" y1="36.485521875" x2="17.878234375" y2="36.09115625" width="0.3048" layer="1"/>
-<wire x1="17.878234375" y1="36.09115625" x2="17.48039375" y2="35.768509375" width="0.3048" layer="1"/>
-<wire x1="17.48039375" y1="35.768509375" x2="17.48039375" y2="35.649609375" width="0.3048" layer="1"/>
+<wire x1="17.8883" y1="36.485521875" x2="17.894615625" y2="36.47920625" width="0.3048" layer="1"/>
+<wire x1="17.8883" y1="36.485521875" x2="17.886653125" y2="35.49869375" width="0.3048" layer="1"/>
 </signal>
 <signal name="N$15">

Commit message: Add files via upload
Parts:
- moved C14 0.20 mm to (17.1, 21.5)
- moved L2 0.07 mm to (15.0, 21.5)
Routing:
- net 18: track 28.7 -> 31.9 mm
- net 19: track 19.0 -> 20.8 mm
- net N$6: track 5.81 -> 7.40 mm, vias 0 -> 3
- net VCC: track 46.5 -> 45.9 mm, vias 10 -> 11
- net RESET: track 5.53 -> 5.23 mm, vias 2 -> 0
- net GND: vias 270 -> 273

Commit message: Add files via upload
Parts:
- IC3: device ok-chips-dev:QFN50P700X700X100-49N -> CC2652R1FRGZT:QFN50P700X700X100-49N
Changed lines of the file:
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@@
 </autorouter>
 <elements>
-<element name="IC3" library="ok-chips-dev" package="QFN50P700X700X100-49N" value="CC2652R1FRGZ" x="13.6758" y="27.6371" smashed="yes" rot="R270">
+<element name="IC3" library="CC2652R1FRGZT" package="QFN50P700X700X100-49N" value="CC2652R1FRGZ" x="13.6758" y="27.6371" smashed="yes" rot="R270">
+<attribute name="ARROW_PART_NUMBER" value="CC2652R1FRGZT" x="13.6758" y="27.6371" size="1.778" layer="27" rot="R270" display="off"/>
+<attribute name="ARROW_PRICE-STOCK" value="https://www.arrow.com/en/products/cc2652r1frgzt/texas-instruments" x="13.6758" y="27.6371" size="1.778" layer="27" rot="R270" display="off"/>
 <attribute name="DESCRIPTION" value="Texas Instruments SimpleLink? Multi-Standard CC2652R Wireless MCU 48-VQFN -40 to 85" x="8.5958" y="-4.1129" size="1.778" layer="27" rot="R270" display="off"/>
 <attribute name="HEIGHT" value="1mm" x="8.5958" y="-4.1129" size="1.778" layer="27" rot="R270" display="off"/>
@@
 <attribute name="MANUFACTURER_PART_NUMBER" value="CC2652R1FRGZT" x="8.5958" y="-4.1129" size="1.778" layer="27" rot="R270" display="off"/>
 <attribute name="MOUSER_PART_NUMBER" value="595-CC2652R1FRGZT" x="8.5958" y="-4.1129" size="1.778" layer="27" rot="R270" display="off"/>
-<attribute name="MOUSER_PRICE-STOCK" value="https://www.mouser.com/Search/Refine.aspx?Keyword=595-CC2652R1FRGZT" x="8.5958" y="-4.1129" size="1.778" layer="27" rot="R270" display="off"/>
+<attribute name="MOUSER_PRICE-STOCK" value="https://www.mouser.co.uk/ProductDetail/Texas-Instruments/CC2652R1FRGZT?qs=rrS6PyfT74ekj88w7n1zLw%3D%3D" x="8.5958" y="-4.1129" size="1.778" layer="27" rot="R270" display="off"/>
 <attribute name="NAME" x="13.6758" y="27.6371" size="0.762" layer="25" font="vector" ratio="10" rot="R90" align="center"/>
-<attribute name="RS_PART_NUMBER" value="" x="8.5958" y="-4.1129" size="1.778" layer="27" rot="R270" display="off"/>
-<attribute name="RS_PRICE-STOCK" value="" x="8.5958" y="-4.1129" size="1.778" layer="27" rot="R270" display="off"/>
 <attribute name="VALUE" x="13.6758" y="27.6371" size="1.27" layer="27" rot="R270" align="center"/>
 </element>
@@
 <attribute name="VALUE" x="22.1010375" y="22.48868125" size="0.6096" layer="27" font="vector" ratio="20" rot="R179.5" align="top-center"/>
 </element>
-<element name="FL1" library="2450BM14G0011T" package="BALUN_2450BM14G0011T" value="2450BM14G0011T" x="16.2" y="33" smashed="yes">
-<attribute name="AVAILABILITY" value="In Stock" x="16.2" y="33" size="1.778" layer="27" display="off"/>
-<attribute name="DESCRIPTION" value=" RF Balun 2.4GHz ~ 2.5GHz 50 / -Ohm 0603 (1608 Metric), 6 PC Pad " x="16.2" y="33" size="1.778" layer="27" display="off"/>
-<attribute name="MF" value="Johanson Technology" x="16.2" y="33" size="1.778" layer="27" display="off"/>
-<attribute name="MP" value="2450BM14G0011T" x="16.2" y="33" size="1.778" layer="27" display="off"/>
-<attribute name="PACKAGE" value="0603 Johanson" x="16.2" y="33" size="1.778" layer="27" display="off"/>
-<attribute name="PRICE" value="None" x="16.2" y="33" size="1.778" layer="27" display="off"/>
-<attribute name="PURCHASE-URL" value="https://pricing.snapeda.com/search/part/2450BM14G0011T/?ref=eda" x="16.2" y="33" size="1.778" layer="27" display="off"/>
-<attribute name="VALUE" x="14.193009375" y="31.494759375" size="0.815265625" layer="27" align="top-left"/>
+<element name="FL1" library="2450BM14G0011T" package="BALUN_2450BM14G0011T" value="2450BM14G0011T" x="16.17239375" y="33.0069" smashed="yes">
+<attribute name="AVAILABILITY" value="In Stock" x="16.17239375" y="33.0069" size="1.778" layer="27" display="off"/>
+<attribute name="DESCRIPTION" value=" RF Balun 2.4GHz ~ 2.5GHz 50 / -Ohm 0603 (1608 Metric), 6 PC Pad " x="16.17239375" y="33.0069" size="1.778" layer="27" display="off"/>
+<attribute name="MF" value="Johanson Technology" x="16.17239375" y="33.0069" size="1.778" layer="27" display="off"/>
+<attribute name="MP" value="2450BM14G0011T" x="16.17239375" y="33.0069" size="1.778" layer="27" display="off"/>
+<attribute name="PACKAGE" value="0603 Johanson" x="16.17239375" y="33.0069" size="1.778" layer="27" display="off"/>
+<attribute name="PRICE" value="None" x="16.17239375" y="33.0069" size="1.778" layer="27" display="off"/>
+<attribute name="PURCHASE-URL" value="https://pricing.snapeda.com/search/part/2450BM14G0011T/?ref=eda" x="16.17239375" y="33.0069" size="1.778" layer="27" display="off"/>
+<attribute name="VALUE" x="14.165403125" y="31.501659375" size="0.815265625" layer="27" align="top-left"/>
 </element>
 <element name="Q1" library="SI2323DS" package="SOT23" value="SI2323DS" x="3.8635" y="18.3175" smashed="yes" rot="R180">
@@
 <via x="0.8873" y="20.3523" extent="1-16" drill="0.3"/>
 <via x="0.8873" y="19.4142" extent="1-16" drill="0.3"/>
-<via x="15.2" y="32.5" extent="1-16" drill="0.2" diameter="0.45"/>
-<via x="15.2" y="33.1" extent="1-16" drill="0.2" diameter="0.45"/>
+<via x="15.144784375" y="32.5" extent="1-16" drill="0.2" diameter="0.45"/>
+<via x="15.137884375" y="33.1" extent="1-16" drill="0.2" diameter="0.45"/>
 <via x="15.2" y="33.9" extent="1-16" drill="0.2" diameter="0.45"/>
 <via x="15.7" y="34.3" extent="1-16" drill="0.2" diameter="0.45"/>
@@
 <contactref element="FL1" pad="4"/>
 <wire x1="16.4258" y1="31.0871" x2="16.4258" y2="31.8258" width="0.254" layer="1"/>
-<wire x1="16.61" y1="32.01" x2="16.61" y2="32.5" width="0.254" layer="1"/>
-<wire x1="16.4258" y1="31.8258" x2="16.61" y2="32.01" width="0.254" layer="1"/>
+<wire x1="16.58239375" y1="31.98239375" x2="16.58239375" y2="32.5069" width="0.254" layer="1"/>
+<wire x1="16.4258" y1="31.8258" x2="16.58239375" y2="31.98239375" width="0.254" layer="1"/>
 </signal>
 <signal name="N$2">
@@
 <contactref element="FL1" pad="3"/>
 <wire x1="15.9258" y1="31.0871" x2="15.9258" y2="31.826165625" width="0.254" layer="1"/>
-<wire x1="15.79" y1="31.961965625" x2="15.79" y2="32.5" width="0.254" layer="1"/>
-<wire x1="15.9258" y1="31.826165625" x2="15.79" y2="31.961965625" width="0.254" layer="1"/>
+<wire x1="15.76239375" y1="31.989571875" x2="15.76239375" y2="32.5069" width="0.254" layer="1"/>
+<wire x1="15.9258" y1="31.826165625" x2="15.76239375" y2="31.989571875" width="0.254" layer="1"/>
 </signal>
 <signal name="1">
@@
 <contactref element="R9" pad="2"/>
 <contactref element="FL1" pad="1"/>
-<wire x1="17.2587125" y1="34.911078125" x2="16.0974375" y2="33.8074375" width="0.3048" layer="1"/>
-<wire x1="15.79" y1="33.5" x2="16.0974375" y2="33.8074375" width="0.3048" layer="1"/>
+<wire x1="17.2587125" y1="34.911078125" x2="16.1404125" y2="33.848278125" width="0.3048" layer="1"/>
+<wire x1="15.76239375" y1="33.5069" x2="16.1404125" y2="33.848278125" width="0.3048" layer="1"/>
 </signal>
 <signal name="N$5">

Commit message: Add files via upload
Parts:
- moved C18 1.23 mm to (18.0, 31.4), turned to 90 degrees
- moved Y1 0.56 mm to (20.4, 30.1)
Routing:
- net VDDR: track 9.74 -> 8.26 mm
- net 3: track 1.07 -> 0.00 mm, vias 1 -> 0
- net 2: track 0.78 -> 0.00 mm, vias 1 -> 0
- net X48M_N: track 3.96 -> 4.48 mm
- net GND: track 1.75 -> 1.68 mm, vias 273 -> 277

Commit message: Add files via upload
Parts:
- moved C3 3.18 mm to (24.0, 23.3), turned to 269.5 degrees
- moved C14 1.71 mm to (18.8, 21.8), turned to 0 degrees
- moved L1 1.22 mm to (8.54, 22.4)
- moved C16 0.99 mm to (11.8, 21.8), turned to 180 degrees
- moved L2 0.41 mm to (15.3, 21.8), turned to 180 degrees
- moved R3 0.29 mm to (24.6, 27.7)
- moved C1 0.23 mm to (8.96, 20.9)
- moved C2 0.23 mm to (8.96, 19.9)
Routing:
- net VDDR: track 8.26 -> 12.4 mm
- net DCDC_SW: track 1.75 -> 3.79 mm
- net VCC: track 45.9 -> 44.0 mm
- net VDDS: track 17.6 -> 19.0 mm
- net GND: vias 277 -> 281
Other:
- board text added: "3V3"
- board text added: "GND"
- board text added: "TCK"
- board text added: "TDI"
- board text added: "TDO"
- board text added: "TMS"
