File: cc2652p_rc4/rc4.brd (EAGLE design)
At the start: 29.2 x 41.8 mm, 45 parts, among them IC3 CC2652R1FRGZ, Q1 SI2323DS, Q2 SI2323DS, Y1 Q22FA12800150, Y2 32.768KHz

Commit message: Add files via upload
Parts:
- IC3: device CC1352P1F3RGZR:RGZ0048A -> CC2652P1FRGZR:RGZ0048A-IPC_B
- moved C3 3.18 mm to (24.0, 23.3), turned to 269.5 degrees
- moved C14 1.71 mm to (18.8, 21.8), turned to 0 degrees
- moved C18 1.23 mm to (18.0, 31.4), turned to 90 degrees
- moved L1 1.22 mm to (8.54, 22.4)
- moved C16 0.99 mm to (11.8, 21.8), turned to 180 degrees
- moved Y1 0.56 mm to (20.4, 30.1)
- moved L2 0.41 mm to (15.3, 21.8), turned to 180 degrees
- moved R3 0.29 mm to (24.6, 27.7)
- moved C1 0.23 mm to (8.96, 20.9)
- moved C2 0.23 mm to (8.96, 19.9)
Connections:
- net X48M_N renamed N$4
- net X48M_P renamed N$21
Routing:
- net VDDR: track 9.84 -> 12.4 mm
- net DCDC_SW: track 1.80 -> 3.79 mm
- net VDDS: track 17.8 -> 18.9 mm
- net VCC: track 45.9 -> 46.9 mm
- net 7: track 5.24 -> 4.67 mm
- net GND: track 1.75 -> 1.68 mm, vias 276 -> 286
Other:
- board text added: "3V3"
- board text added: "GND"
- board text added: "TCK"
- board text added: "TDI"
- board text added: "TDO"
- board text added: "TMS"

Commit message: Add files via upload
Other:
- board size 29.2 x 41.8 mm -> 29.2 x 41.7 mm
Changed lines of the file:
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@@
 <text x="18.606215625" y="5.0889625" size="0.8128" layer="25" rot="R180">JLCJLCJLCJLC</text>
 <hole x="26.076" y="5.888" drill="1.8"/>
-<wire x1="29.4" y1="0.2405" x2="0.2" y2="0.2405" width="0.1524" layer="20"/>
-<wire x1="0.2" y1="0.2405" x2="0.2" y2="26.8" width="0.1524" layer="20"/>
-<wire x1="29.4" y1="0.2405" x2="29.4" y2="27" width="0.1524" layer="20"/>
+<wire x1="0.2" y1="0.3" x2="0.2" y2="26.8" width="0.1524" layer="20"/>
 <hole x="4.776" y="37.388" drill="1.8"/>
+<wire x1="29.4" y1="0.3" x2="29.4" y2="27" width="0.1524" layer="20"/>
 <wire x1="6.3" y1="42" x2="23.3" y2="42" width="0.1524" layer="20"/>
 <wire x1="23.3" y1="42" x2="23.7" y2="42" width="0.1524" layer="20"/>
@@
 <text x="1.480896875" y="27.173084375" size="0.8128" layer="26" font="vector" ratio="12" rot="MR179.6">GND</text>
 <text x="1.480896875" y="25.873084375" size="0.8128" layer="26" font="vector" ratio="12" rot="MR179.6">3V3</text>
+<wire x1="16.2" y1="3.4" x2="22.3" y2="0.4" width="0.1524" layer="20" curve="-37.725056"/>
+<wire x1="22.3" y1="0.4" x2="22.4" y2="0.3" width="0.1524" layer="20" curve="0.101255"/>
+<wire x1="7.4" y1="0.3" x2="0.2" y2="0.3" width="0.1524" layer="20"/>
+<wire x1="22.4" y1="0.3" x2="29.4" y2="0.3" width="0.1524" layer="20"/>
+<wire x1="16.2" y1="3.4" x2="7.4" y2="0.3" width="0.1524" layer="20" curve="53.463074"/>
 </plain>
 <attributes>
@@
 </element>
 <element name="C1" library="ok-discretes-dev" package="_PKG_C_0402" value="100n" x="8.96473125" y="20.8927625" smashed="yes">
-<attribute name="NAME" x="7.001528125" y="20.813421875" size="0.762" layer="25" font="vector" ratio="10"/>
+<attribute name="NAME" x="6.901528125" y="20.613421875" size="0.762" layer="25" font="vector" ratio="10"/>
 <attribute name="VALUE" x="8.07573125" y="19.8767625" size="0.508" layer="27" font="vector"/>
 </element>
 <element name="C2" library="ok-discretes-dev" package="_PKG_C_0402" value="100n" x="8.96473125" y="19.8640625" smashed="yes">
-<attribute name="NAME" x="8.44735" y="18.57955" size="0.762" layer="25" font="vector" ratio="10"/>
+<attribute name="NAME" x="6.84735" y="19.57955" size="0.762" layer="25" font="vector" ratio="10"/>
 <attribute name="VALUE" x="8.07573125" y="18.8480625" size="0.508" layer="27" font="vector"/>
 </element>
@@
 </element>
 <element name="C11" library="ok-discretes-dev" package="_PKG_C_0402" value="100n" x="8.2259" y="30.3803" smashed="yes" rot="R180">
-<attribute name="NAME" x="7.2514" y="30.7723" size="0.762" layer="25" font="vector" ratio="10" rot="R180"/>
+<attribute name="NAME" x="9.0514" y="31.6723" size="0.762" layer="25" font="vector" ratio="10" rot="R180"/>
 <attribute name="VALUE" x="9.1149" y="31.3963" size="0.762" layer="27" font="vector" ratio="10" rot="R180"/>
 </element>
@@
 <via x="6.2032" y="0.9649" extent="1-16" drill="0.3"/>
 <via x="7.1413" y="0.9649" extent="1-16" drill="0.3"/>
-<via x="8.0794" y="0.9649" extent="1-16" drill="0.3"/>
-<via x="9.0175" y="0.9649" extent="1-16" drill="0.3"/>
-<via x="9.9556" y="0.9649" extent="1-16" drill="0.3"/>
-<via x="10.8937" y="0.9649" extent="1-16" drill="0.3"/>
-<via x="11.8318" y="0.9649" extent="1-16" drill="0.3"/>
-<via x="12.7699" y="0.9649" extent="1-16" drill="0.3"/>
-<via x="13.708" y="0.9649" extent="1-16" drill="0.3"/>
-<via x="14.6461" y="0.9649" extent="1-16" drill="0.3"/>
-<via x="15.5842" y="0.9649" extent="1-16" drill="0.3"/>
-<via x="16.5223" y="0.9649" extent="1-16" drill="0.3"/>
-<via x="17.4604" y="0.9649" extent="1-16" drill="0.3"/>
-<via x="18.3985" y="0.9649" extent="1-16" drill="0.3"/>
-<via x="19.3366" y="0.9649" extent="1-16" drill="0.3"/>
-<via x="20.2747" y="0.9649" extent="1-16" drill="0.3"/>
-<via x="21.2128" y="0.9649" extent="1-16" drill="0.3"/>
-<via x="22.1509" y="0.9649" extent="1-16" drill="0.3"/>
+<via x="7.8794" y="1.4649" extent="1-16" drill="0.3"/>
+<via x="8.7175" y="2.0649" extent="1-16" drill="0.3"/>
+<via x="9.4556" y="2.5649" extent="1-16" drill="0.3"/>
+<via x="10.3937" y="3.0649" extent="1-16" drill="0.3"/>
+<via x="11.4318" y="3.4649" extent="1-16" drill="0.3"/>
+<via x="12.3699" y="3.7649" extent="1-16" drill="0.3"/>
+<via x="13.308" y="3.9649" extent="1-16" drill="0.3"/>
+<via x="14.2461" y="4.0649" extent="1-16" drill="0.3"/>
+<via x="15.4842" y="4.0649" extent="1-16" drill="0.3"/>
+<via x="16.4223" y="3.9649" extent="1-16" drill="0.3"/>
+<via x="17.5604" y="3.6649" extent="1-16" drill="0.3"/>
+<via x="18.5985" y="3.3649" extent="1-16" drill="0.3"/>
+<via x="19.6366" y="2.9649" extent="1-16" drill="0.3"/>
+<via x="20.5747" y="2.4649" extent="1-16" drill="0.3"/>
+<via x="21.4128" y="1.9649" extent="1-16" drill="0.3"/>
+<via x="22.1351" y="1.2509" extent="1-16" drill="0.3"/>
 <via x="23.089" y="0.9649" extent="1-16" drill="0.3"/>
 <via x="24.0271" y="0.9649" extent="1-16" drill="0.3"/>
@@
 <contactref element="IC3" pad="1"/>
 <contactref element="FL1" pad="4"/>
-<wire x1="16.4258" y1="31.138346875" x2="16.4258" y2="31.8258" width="0.254" layer="1"/>
-<wire x1="16.58239375" y1="31.98239375" x2="16.58239375" y2="32.5069" width="0.254" layer="1"/>
-<wire x1="16.4258" y1="31.8258" x2="16.58239375" y2="31.98239375" width="0.254" layer="1"/>
+<wire x1="16.4258" y1="31.138346875" x2="16.4295" y2="31.652496875" width="0.3048" layer="1"/>
+<wire x1="16.4295" y1="31.652496875" x2="16.58239375" y2="32.5069" width="0.3048" layer="1"/>
 </signal>
 <signal name="N$2">
 <contactref element="IC3" pad="2"/>
 <contactref element="FL1" pad="3"/>
-<wire x1="15.9258" y1="31.138346875" x2="15.9258" y2="31.826165625" width="0.254" layer="1"/>
-<wire x1="15.76239375" y1="31.989571875" x2="15.76239375" y2="32.5069" width="0.254" layer="1"/>
-<wire x1="15.9258" y1="31.826165625" x2="15.76239375" y2="31.989571875" width="0.254" layer="1"/>
+<wire x1="15.9258" y1="31.138346875" x2="15.92864375" y2="31.65359375" width="0.3048" layer="1"/>
+<wire x1="15.92864375" y1="31.65359375" x2="15.76239375" y2="32.5069" width="0.3048" layer="1"/>
 </signal>
 <signal name="5">

Commit message: Add files via upload
Parts:
- added C4, C9: 6p8, ok-discretes-dev:_PKG_C_0402
Connections:
- net GND: now also C4.1, C9.1
- net N$21: now also C9.2
- net N$4: now also C4.2
Routing:
- net N$21: track 3.03 -> 4.89 mm
- net N$4: track 4.39 -> 6.01 mm
- net GND: vias 286 -> 284
Changed lines of the file:
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@@
 <param name="mvStopFrame" value="1"/>
 <param name="mvCreamFrame" value="0"/>
-<param name="mlMinStopFrame" value="2.5mil"/>
-<param name="mlMaxStopFrame" value="2.5mil"/>
+<param name="mlMinStopFrame" value="2mil"/>
+<param name="mlMaxStopFrame" value="2mil"/>
 <param name="mlMinCreamFrame" value="0mil"/>
 <param name="mlMaxCreamFrame" value="0mil"/>
@@
 <attribute name="MFG_NAME" value="KYOCERA" x="20.39691875" y="30.0895625" size="1.778" layer="27" rot="R270" display="off"/>
 <attribute name="MFG_PART" value="CX2016DB48000C0FPLC1" x="20.39691875" y="30.0895625" size="1.778" layer="27" rot="R270" display="off"/>
-<attribute name="NAME" x="22.42359375" y="29.547875" size="0.762" layer="25" font="vector" ratio="10" rot="R90"/>
+<attribute name="NAME" x="18.93710625" y="29.53355625" size="0.762" layer="25" font="vector" ratio="10" rot="R90"/>
 <attribute name="VALUE" x="17.85691875" y="31.3595625" size="0.762" layer="27" font="vector" ratio="10" rot="R270"/>
 </element>
@@
 <attribute name="TP_SIGNAL_NAME" value="" x="2.4" y="24.965709375" size="1" layer="37"/>
 <attribute name="VALUE" x="1.892" y="26.362709375" size="0.0254" layer="27"/>
+</element>
+<element name="C9" library="ok-discretes-dev" package="_PKG_C_0402" value="6p8" x="21.43494375" y="32.155446875" smashed="yes" rot="R180">
+<attribute name="NAME" x="23.441021875" y="32.57991875" size="0.762" layer="25" font="vector" rot="R180"/>
+<attribute name="VALUE" x="22.32394375" y="33.171446875" size="0.508" layer="27" font="vector" rot="R180"/>
+</element>
+<element name="C4" library="ok-discretes-dev" package="_PKG_C_0402" value="6p8" x="22.593621875" y="29.785778125" smashed="yes" rot="R270">
+<attribute name="NAME" x="22.135128125" y="30.734421875" size="0.762" layer="25" font="vector"/>
+<attribute name="VALUE" x="21.577621875" y="30.674778125" size="0.508" layer="27" font="vector" rot="R270"/>
 </element>
 </elements>
@@
 <via x="27.7" y="27.1" extent="1-16" drill="0.2" diameter="0.45"/>
 <via x="26.9" y="28" extent="1-16" drill="0.2" diameter="0.45"/>
-<via x="22.4" y="31.6" extent="1-16" drill="0.2" diameter="0.45"/>
 <via x="26.4" y="26" extent="1-16" drill="0.2" diameter="0.45"/>
 <via x="27.7" y="24.6" extent="1-16" drill="0.2" diameter="0.45"/>
@@
 <via x="26.6" y="23.3" extent="1-16" drill="0.2" diameter="0.45"/>
 <via x="25.1552875" y="23.77158125" extent="1-16" drill="0.2" diameter="0.45"/>
-<via x="22.7" y="29" extent="1-16" drill="0.2" diameter="0.45"/>
 <via x="22.8" y="27.5" extent="1-16" drill="0.2" diameter="0.45"/>
 <via x="20.7" y="28.4" extent="1-16" drill="0.2" diameter="0.45"/>
-<via x="20.9" y="31.8" extent="1-16" drill="0.2" diameter="0.45"/>
 <via x="5.7" y="23.3" extent="1-16" drill="0.2" diameter="0.45"/>
 <via x="5.9" y="20.1" extent="1-16" drill="0.2" diameter="0.45"/>
@@
 <via x="17.01600625" y="22.51929375" extent="1-16" drill="0.2" diameter="0.45"/>
 <via x="13.5490125" y="22.5467" extent="1-16" drill="0.2" diameter="0.45"/>
+<contactref element="C9" pad="1"/>
+<contactref element="C4" pad="1"/>
+<via x="19.308884375" y="31.7607125" extent="1-16" drill="0.2" diameter="0.45"/>
 </signal>
 <signal name="DCOUPL">
@@
 <wire x1="20.97191875" y1="29.40193125" x2="20.307534375" y2="30.066315625" width="0.1524" layer="1"/>
 <wire x1="18.823328125" y1="30.066315625" x2="20.307534375" y2="30.066315625" width="0.1524" layer="1"/>
+<contactref element="C4" pad="2"/>
+<wire x1="20.97191875" y1="29.3645625" x2="22.5848375" y2="29.3645625" width="0.1524" layer="1"/>
+<wire x1="22.5848375" y1="29.3645625" x2="22.593621875" y2="29.355778125" width="0.1524" layer="1"/>
 </signal>
 <signal name="N$21">
 <contactref element="IC3" pad="47"/>
+<contactref element="C9" pad="2"/>
 <contactref element="Y1" pad="1"/>
-<wire x1="17.177046875" y1="29.8871" x2="18.189715625" y2="29.8871" width="0.1524" layer="1"/>
-<wire x1="18.189715625" y1="29.8871" x2="19.119990625" y2="30.817375" width="0.1524" layer="1"/>
-<wire x1="19.119990625" y1="30.817375" x2="19.81910625" y2="30.817375" width="0.1524" layer="1"/>
-<wire x1="19.81910625" y1="30.817375" x2="19.82191875" y2="30.8145625" width="0.1524" layer="1"/>
+<wire x1="18.248975" y1="29.8871" x2="18.70759375" y2="30.34571875" width="0.1524" layer="1"/>
+<wire x1="17.177046875" y1="29.8871" x2="18.248975" y2="29.8871" width="0.1524" layer="1"/>
+<wire x1="21.00494375" y1="32.03495625" x2="19.82191875" y2="30.85193125" width="0.1524" layer="1"/>
+<wire x1="19.82191875" y1="30.85193125" x2="19.82191875" y2="30.8145625" width="0.1524" layer="1"/>
+<wire x1="21.00494375" y1="32.155446875" x2="21.00494375" y2="32.03495625" width="0.1524" layer="1"/>
+<wire x1="19.82191875" y1="30.766271875" x2="19.82191875" y2="30.8145625" width="0.1524" layer="1"/>
+<wire x1="19.82191875" y1="30.766271875" x2="19.401365625" y2="30.34571875" width="0.1524" layer="1"/>
+<wire x1="18.70759375" y1="30.34571875" x2="19.401365625" y2="30.34571875" width="0.1524" layer="1"/>
 </signal>
 </signals>
