File: cc2652p_rc4/v1.1/rc4.1_1.brd (EAGLE design)
At the start: 29.2 x 41.8 mm, 53 parts, among them IC3 CC2652R1FRGZ, Q1 SI2323DS, Q2 SI2323DS, Y1 Q22FA12800150, Y2 32.768KHz

Commit message: Add files via upload
Parts:
- added C21, C22: 7.5p, ok-discretes-dev:_PKG_C_0402
- moved C20 0.08 mm to (19.6, 34.6)
Connections:
- net GND: now also C21.1, C22.1
- net N$21: now also C21.2
- net N$4: now also C22.2
Routing:
- net N$21: track 3.37 -> 5.11 mm
- net N$4: track 4.70 -> 6.32 mm
- net GND: vias 283 -> 285
Other:
- board size 29.2 x 41.8 mm -> 29.2 x 41.6 mm

Commit message: Add files via upload
Parts:
- added C24, C25, C26, C27: 100n, ok-discretes-dev:_PKG_C_0402
- C10, C19: value CAP0402 -> 1pF
- C21, C22: value 7.5p -> 6.8p
- C23: value 1.8p -> 1.8pF
- C4: value CAP0402 -> 1pf
- C9: value CAP0402 -> 12pF
- L3, L4: value IND0402IND0402 -> 2.4nH
- L5, L6: value IND0402IND0402 -> 2nH
Connections:
- net 18: now also C26.1
- net 19: now also C25.1
- net 21: now also C27.1
- net 5: now also C24.1
- net GND: now also C24.2, C25.2, C26.2, C27.2
Routing:
- net 19: track 20.7 -> 22.8 mm
- net 21: track 13.7 -> 15.2 mm
- net 5: track 10.9 -> 12.2 mm
- net TCK: track 14.4 -> 15.5 mm
- net 18: track 31.9 -> 32.6 mm
- net TMS: track 14.5 -> 15.1 mm
- net GND: vias 285 -> 283
