File: cc2652p_rc4/v1.1/rc4.1_1.brd (EAGLE design)
At the start: 29.2 x 41.6 mm, 59 parts, among them IC3 CC2652R1FRGZ, Q1 SI2323DS, Q2 SI2323DS, Y1 Q22FA12800150, Y2 32.768KHz

Commit message: Add files via upload
Parts:
- added TP3, TP4: TPB2,54, testpad:B2,54
Connections:
- net GND: now also TP3.TP
- net N$6: now also TP4.TP
Routing:
- net N$6: track 7.40 -> 18.1 mm, vias 3 -> 4
- net 18: track 32.6 -> 30.6 mm
Changed lines of the file:
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@@
 <drawing>
 <settings>
-<setting alwaysvectorfont="no"/>
+<setting alwaysvectorfont="yes"/>
 <setting verticaltext="up"/>
 </settings>
@@
 <wire x1="0.8" y1="36.8" x2="0.2" y2="26.8" width="0.1524" layer="20"/>
 <wire x1="28.7" y1="36.7" x2="29.4" y2="27" width="0.1524" layer="20"/>
-<text x="2.2401875" y="1.36555" size="1.016" layer="25" font="vector" ratio="12" rot="SR89.6">t.me/deaxx</text>
+<text x="1.639353125" y="1.529053125" size="1.27" layer="26" font="vector" ratio="12" rot="SMR89.6">t.me/deaxx</text>
 <wire x1="5.7" y1="14" x2="24" y2="14" width="0.1524" layer="21"/>
 <wire x1="5.7" y1="14" x2="5.8" y2="14.1" width="0.1524" layer="25"/>
@@
 <attribute name="VALUE" x="27.02265" y="26.22498125" size="0.508" layer="27" font="vector" rot="R90"/>
 </element>
+<element name="TP3" library="testpad" library_urn="urn:adsk.eagle:library:385" package="B2,54" package3d_urn="urn:adsk.eagle:package:27948/1" value="TPB2,54" x="26.957303125" y="2.717915625" smashed="yes">
+<attribute name="POPULARITY" value="3" x="26.957303125" y="2.717915625" size="1.778" layer="27" display="off"/>
+<attribute name="TP_SIGNAL_NAME" value="" x="26.957303125" y="2.717915625" size="1.778" layer="27" display="off"/>
+<attribute name="VALUE" x="25.687303125" y="1.320915625" size="0.0254" layer="27"/>
+</element>
+<element name="TP4" library="testpad" library_urn="urn:adsk.eagle:library:385" package="B2,54" package3d_urn="urn:adsk.eagle:package:27948/1" value="TPB2,54" x="2.623946875" y="2.63589375" smashed="yes">
+<attribute name="POPULARITY" value="3" x="2.623946875" y="2.63589375" size="1.778" layer="27" display="off"/>
+<attribute name="TP_SIGNAL_NAME" value="" x="2.623946875" y="2.63589375" size="1.778" layer="27" display="off"/>
+<attribute name="VALUE" x="1.353946875" y="1.23889375" size="0.0254" layer="27"/>
+</element>
 </elements>
 <signals>
@@
 <contactref element="C25" pad="2"/>
 <contactref element="C27" pad="2"/>
+<contactref element="TP3" pad="TP"/>
 </signal>
 <signal name="DCOUPL">
@@
 <wire x1="7.7" y1="25.7" x2="7.7" y2="27.2" width="0.1524" layer="16"/>
 <wire x1="7.7" y1="27.2" x2="7.3" y2="27.6" width="0.1524" layer="16"/>
-<wire x1="3.1" y1="29.4" x2="2.4" y2="29.4" width="0.1524" layer="16"/>
+<wire x1="4.1513125" y1="28.3914375" x2="3.451203125" y2="28.3914375" width="0.1524" layer="16"/>
+<wire x1="3.451203125" y1="28.3914375" x2="2.442640625" y2="29.4" width="0.1524" layer="16"/>
+<wire x1="2.442640625" y1="29.4" x2="2.4" y2="29.4" width="0.1524" layer="16"/>
 <wire x1="10.149784375" y1="23.250215625" x2="7.7" y2="25.7" width="0.1524" layer="16"/>
-<wire x1="7.3" y1="27.6" x2="4.9" y2="27.6" width="0.1524" layer="16"/>
-<wire x1="4.9" y1="27.6" x2="3.1" y2="29.4" width="0.1524" layer="16"/>
+<wire x1="7.3" y1="27.6" x2="4.94275" y2="27.6" width="0.1524" layer="16"/>
+<wire x1="4.94275" y1="27.6" x2="4.1513125" y2="28.3914375" width="0.1524" layer="16"/>
 <contactref element="IC3" pad="26"/>
 <wire x1="11.4258" y1="24.135853125" x2="11.4258" y2="23.543584375" width="0.1524" layer="1"/>
@@
 <wire x1="12.184228125" y1="17.119" x2="13.585828125" y2="18.5206" width="0.1524" layer="16"/>
 <wire x1="20.766175" y1="18.5206" x2="21.748228125" y2="17.538546875" width="0.1524" layer="16"/>
-<wire x1="21.748228125" y1="17.538546875" x2="21.748228125" y2="14.950215625" width="0.1524" layer="16"/>
-<wire x1="21.748228125" y1="14.950215625" x2="22.487784375" y2="14.210659375" width="0.1524" layer="16"/>
-<wire x1="22.487784375" y1="14.210659375" x2="27.141159375" y2="14.210659375" width="0.1524" layer="16"/>
+<wire x1="21.748228125" y1="17.538546875" x2="21.748228125" y2="16.1539875" width="0.1524" layer="16"/>
+<wire x1="21.748228125" y1="16.1539875" x2="22.635325" y2="15.266890625" width="0.1524" layer="16"/>
+<wire x1="22.635325" y1="15.266890625" x2="27.5" y2="15.266890625" width="0.1524" layer="16"/>
 <wire x1="13.585828125" y1="18.5206" x2="20.766175" y2="18.5206" width="0.1524" layer="16"/>
 <via x="27.5" y="15.3" extent="1-16" drill="0.2" diameter="0.45"/>
 <wire x1="27.5" y1="16.35" x2="27.5" y2="15.3" width="0.1524" layer="1"/>
-<wire x1="27.5" y1="14.5695" x2="27.5" y2="15.3" width="0.1524" layer="16"/>
-<wire x1="27.141159375" y1="14.210659375" x2="27.5" y2="14.5695" width="0.1524" layer="16"/>
+<wire x1="27.5" y1="15.266890625" x2="27.5" y2="15.3" width="0.1524" layer="16"/>
 <contactref element="IC3" pad="28"/>
 <wire x1="12.4258" y1="23.5258" x2="12.4258" y2="24.135853125" width="0.1524" layer="1"/>
@@
 <wire x1="3.8873" y1="11.414" x2="3.8873" y2="12.2" width="0.4064" layer="1"/>
 <wire x1="3.9" y1="11.5" x2="3.9" y2="12.2" width="0.4064" layer="1"/>
-<wire x1="3.9" y1="10.7" x2="3.9" y2="11.5" width="0.4064" layer="1"/>
+<wire x1="3.9" y1="10.7" x2="3.9" y2="11.44051875" width="0.4064" layer="1"/>
+<wire x1="3.9" y1="11.44051875" x2="3.9" y2="11.5" width="0.4064" layer="1"/>
 <wire x1="3.8873" y1="11.414" x2="3.8873" y2="11.4873" width="0.4064" layer="1"/>
 <wire x1="3.9" y1="11.5" x2="3.8873" y2="11.4873" width="0.4064" layer="1"/>
+<contactref element="TP4" pad="TP"/>
+<wire x1="2.623946875" y1="2.63589375" x2="2.623946875" y2="5.7522625" width="0.254" layer="1"/>
+<wire x1="2.623946875" y1="5.7522625" x2="1.891434375" y2="6.484775" width="0.254" layer="1"/>
+<wire x1="1.891434375" y1="6.484775" x2="1.891434375" y2="10.64275" width="0.254" layer="1"/>
+<wire x1="2.689203125" y1="11.44051875" x2="3.9" y2="11.44051875" width="0.254" layer="1"/>
+<wire x1="1.891434375" y1="10.64275" x2="2.689203125" y2="11.44051875" width="0.254" layer="1"/>
+<via x="2.63659375" y="2.61971875" extent="1-16" drill="0.25"/>
+<wire x1="2.623946875" y1="2.63589375" x2="2.63659375" y2="2.623246875" width="0.1524" layer="1"/>
+<wire x1="2.63659375" y1="2.623246875" x2="2.63659375" y2="2.61971875" width="0.1524" layer="1"/>
 </signal>
 <signal name="N$11">
