File: cc2652p_rc4/v1.1/rc4.1_1.sch (EAGLE design)
At the start: 53 parts, among them IC3 CC2652R1FRGZ, Q1 SI2323DS, Q2 SI2323DS, Y1 Q22FA12800150, Y2 32.768KHz

Commit message: Add files via upload
Parts:
- added C21, C22: 7.5p, ok-discretes-dev:CAP-0402
Connections:
- net GND: now also C21.1, C22.1
- net N$21: now also C21.2
- net N$4: now also C22.2
Other:
- moved on the sheet: GND, R2, R3, R4, R5, S1, S2, S3, S4, TCK, TDI, TDO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

Commit message: Add files via upload
Parts:
- added C24, C25, C26, C27: 100n, ok-discretes-dev:CAP-0402
- C10, C19: value CAP0402 -> 1pF
- C21, C22: value 7.5p -> 6.8p
- C23: value 1.8p -> 1.8pF
- C4: value CAP0402 -> 1pf
- C9: value CAP0402 -> 12pF
- L3, L4: value IND0402IND0402 -> 2.4nH
- L5, L6: value IND0402IND0402 -> 2nH
Connections:
- net 18: now also C26.1
- net 19: now also C25.1
- net 21: now also C27.1
- net 5: now also C24.1
- net GND: now also C24.2, C25.2, C26.2, C27.2
Other:
- moved on the sheet: GND, TCK, TDI, TDO, TMS, VCC

Commit message: Add files via upload
Parts:
- added TP3, TP4: TPB2,54, testpad:TPB2,54
Connections:
- net GND: now also TP3.TP
- net N$6: now also TP4.TP
Changed lines of the file:
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@@
 <part name="GND27" library="supply1" library_urn="urn:adsk.eagle:library:371" deviceset="GND" device=""/>
 <part name="GND30" library="supply1" library_urn="urn:adsk.eagle:library:371" deviceset="GND" device=""/>
+<part name="TP3" library="testpad" library_urn="urn:adsk.eagle:library:385" deviceset="TP" device="B2,54" package3d_urn="urn:adsk.eagle:package:27948/1"/>
+<part name="TP4" library="testpad" library_urn="urn:adsk.eagle:library:385" deviceset="TP" device="B2,54" package3d_urn="urn:adsk.eagle:package:27948/1"/>
 </parts>
 <sheets>
@@
 <instance part="GND30" gate="1" x="121.92" y="5.08" smashed="yes">
 <attribute name="VALUE" x="119.38" y="2.54" size="1.778" layer="96"/>
+</instance>
+<instance part="TP3" gate="G$1" x="22.86" y="20.32" smashed="yes" rot="R180">
+<attribute name="NAME" x="24.13" y="19.05" size="1.778" layer="95" rot="R180"/>
+<attribute name="TP_SIGNAL_NAME" x="21.59" y="21.59" size="1.778" layer="97" rot="R180"/>
+</instance>
+<instance part="TP4" gate="G$1" x="7.62" y="43.18" smashed="yes">
+<attribute name="NAME" x="6.35" y="44.45" size="1.778" layer="95"/>
+<attribute name="TP_SIGNAL_NAME" x="8.89" y="41.91" size="1.778" layer="97"/>
 </instance>
 </instances>
@@
 <pinref part="Q2" gate="G$1" pin="G"/>
 <wire x1="35.56" y1="25.4" x2="35.56" y2="33.02" width="0.1524" layer="91"/>
+<pinref part="TP3" gate="G$1" pin="TP"/>
+<wire x1="22.86" y1="22.86" x2="22.86" y2="25.4" width="0.1524" layer="91"/>
 </segment>
 <segment>
@@
 <pinref part="Q1" gate="G$1" pin="D"/>
 <wire x1="7.62" y1="38.1" x2="15.24" y2="38.1" width="0.1524" layer="91"/>
-</segment>
-</net>
+<pinref part="TP4" gate="G$1" pin="TP"/>
+<wire x1="7.62" y1="40.64" x2="7.62" y2="38.1" width="0.1524" layer="91"/>
+<junction x="7.62" y="38.1"/>
+</segment>
+</net>
